File: sha2017_rev0_1_0_dev.sch (EAGLE design)
At the start: 116 parts, among them IC1 AP7215, IC2 CPT112, IC3 CP210X_USB_UART, IC4 ESP32WROOM32, IC5 MCP73833, IC6 FXL6408, M1 MOTOR10MM, Q1 MMBT2222A, Q2 MMBT2222A, Q3 SI1304 BDL, Q4 MOSFET-PCHANNEL, Q5 MMBT2222A, Q6 MOSFET-PCHANNEL, Q7 MMBT2222A, Q8 MMBT2222A, T1 SI2301DS, X1_ JST-PH3, X701 2908-05WB-MG

Commit message: placed most of the parts
Parts:
- removed GND, SIG, VDD: (no value), wirepad:SMD2
- removed JP1: M05X2SHD_SMD, SparkFun-Connectors:M05X2SHD_SMD
- removed M1: MOTOR10MM, SparkFun-Electromechanical:MOTOR10MM
- added J2: (no value), EAGLE-BOARD-TO-BOARD_CONNECTORS-rev16c:610X12243021
- added R27, R28: 470R, rcl:R-EU_R0603
- added U$1: MOTOR10MM, badge:MOTOR10MM
Connections:
- removed net N$44: M1.+, R12.1
- removed net WS2812_POWER1: R11.1
- new net N$16: Q7.C, U$1.-
- new net WS2812_DATA_OUT: D9.DOUT, J2.8
- new net WS2812_POWER_EN: IC6.GPIO0, R11.1, R18.1
- net +3V3: now also R27.1, R28.1
- net 3V3_SWITCHED: now also J2.1; no longer JP1.1
- net EXTIO-0: now also IC4.IO33, J2.3; no longer IC4.IO35, JP1.3
- net EXTIO-1: now also J2.4; no longer JP1.5
- net EXTIO-2: now also J2.5; no longer JP1.7
- net EXTIO-3: now also J2.9; no longer JP1.8
- net EXTIO-4: now also J2.10; no longer JP1.6
- net EXTIO-5: now also J2.11; no longer JP1.4
- net GND: now also J2.12; no longer GND.P, JP1.2, JP1.9
- net I2C_SCL: now also J2.7, R27.2
- net I2C_SDA: now also J2.6, R28.2
- net N$18: now also R12.1, U$1.+; no longer M1.-, Q7.C
- net VBAT: no longer R12.2
- net VBAT_SENSE: now also IC4.IO35; no longer IC4.IO33
- net VCC: now also R12.2
- net VUSB_SENSE: now also IC4.IO34; no longer IC4.IO32
- net WS2812_DATA: now also IC4.IO32; no longer IC4.IO34, SIG.P
- net WS2812_POWER: now also J2.2; no longer IC6.GPIO0, JP1.10, R18.1, VDD.P

Commit message: finised routing
Parts:
- added S1, S2: SWITCH-MOMENTARY-2SMD, SparkFun-Electromechanical:SWITCH-MOMENTARY-2SMD
- renumbered J2 to J3
Connections:
- net CHRG_STAT: now also IC6.GPIO0; no longer IC6.GPIO4
- net ESP32_!RESET: now also S2.2
- net ESP32_FLASH/TOUCHE_MENU: now also S1.2
- net EXTIO-0: now also J3.10; no longer J3.3
- net EXTIO-1: now also J3.9; no longer J3.4
- net EXTIO-2: now also J3.8; no longer J3.5
- net EXTIO-3: now also IC6.GPIO7, J3.4; no longer IC6.GPIO5, J3.9
- net EXTIO-4: now also J3.3; no longer J3.10
- net EXTIO-5: now also IC6.GPIO5, J3.2; no longer IC6.GPIO7, J3.11
- net GND: now also S1.1, S2.1
- net SD_CD: now also IC6.GPIO4; no longer IC6.GPIO2
- net WS2812_DATA_OUT: now also J3.5; no longer J3.8
- net WS2812_POWER: now also J3.11; no longer J3.2
- net WS2812_POWER_EN: now also IC6.GPIO2; no longer IC6.GPIO0
Changed lines of the file:
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@@
 <part name="+2V4" library="supply1" deviceset="+3V3" device=""/>
 <part name="+2V5" library="supply1" deviceset="+3V3" device=""/>
-<part name="J2" library="EAGLE-BOARD-TO-BOARD_CONNECTORS-rev16c" deviceset="610X12243021" device=""/>
+<part name="S1" library="SparkFun-Electromechanical" deviceset="SWITCH-MOMENTARY-2" device="SMD"/>
+<part name="S2" library="SparkFun-Electromechanical" deviceset="SWITCH-MOMENTARY-2" device="SMD"/>
+<part name="GND60" library="supply1" deviceset="GND" device=""/>
+<part name="J3" library="EAGLE-BOARD-TO-BOARD_CONNECTORS-rev16c" deviceset="610X12243021" device=""/>
 </parts>
 <sheets>
@@
 <instance part="U$1" gate="G$1" x="271.78" y="63.5"/>
 <instance part="P+7" gate="VCC" x="271.78" y="83.82"/>
+<instance part="S1" gate="G$1" x="177.8" y="154.94"/>
+<instance part="S2" gate="G$1" x="177.8" y="147.32"/>
+<instance part="GND60" gate="1" x="170.18" y="142.24"/>
 </instances>
 <busses>
@@
 <pinref part="C37" gate="G$1" pin="2"/>
 <pinref part="GND57" gate="1" pin="GND"/>
+</segment>
+<segment>
+<pinref part="S1" gate="G$1" pin="1"/>
+<wire x1="172.72" y1="154.94" x2="170.18" y2="154.94" width="0.1524" layer="91"/>
+<wire x1="170.18" y1="154.94" x2="170.18" y2="147.32" width="0.1524" layer="91"/>
+<pinref part="S2" gate="G$1" pin="1"/>
+<wire x1="170.18" y1="147.32" x2="170.18" y2="144.78" width="0.1524" layer="91"/>
+<wire x1="170.18" y1="147.32" x2="172.72" y2="147.32" width="0.1524" layer="91"/>
+<junction x="170.18" y="147.32"/>
+<pinref part="GND60" gate="1" pin="GND"/>
 </segment>
 </net>
@@
 <label x="205.74" y="198.12" size="1.27" layer="95" xref="yes"/>
 </segment>
+<segment>
+<wire x1="182.88" y1="147.32" x2="187.96" y2="147.32" width="0.1524" layer="91"/>
+<label x="187.96" y="147.32" size="1.27" layer="95" xref="yes"/>
+<pinref part="S2" gate="G$1" pin="2"/>
+</segment>
 </net>
 <net name="ESP32_FLASH/TOUCHE_MENU" class="0">
@@
 <wire x1="198.12" y1="167.64" x2="200.66" y2="167.64" width="0.1524" layer="91"/>
 <junction x="200.66" y="167.64"/>
+</segment>
+<segment>
+<wire x1="182.88" y1="154.94" x2="187.96" y2="154.94" width="0.1524" layer="91"/>
+<label x="187.96" y="154.94" size="1.27" layer="95" xref="yes"/>
+<pinref part="S1" gate="G$1" pin="2"/>
 </segment>
 </net>
@@
 <instance part="+2V4" gate="G$1" x="142.24" y="88.9"/>
 <instance part="+2V5" gate="G$1" x="134.62" y="91.44"/>
-<instance part="J2" gate="G$1" x="274.32" y="63.5"/>
+<instance part="J3" gate="G$1" x="274.32" y="63.5"/>
 </instances>
 <busses>
@@
 <wire x1="302.26" y1="68.58" x2="302.26" y2="66.04" width="0.1524" layer="91"/>
 <pinref part="GND61" gate="1" pin="GND"/>
-<pinref part="J2" gate="G$1" pin="12"/>
+<pinref part="J3" gate="G$1" pin="12"/>
 </segment>
 </net>
@@
 <net name="SD_CD" class="0">
 <segment>
-<label x="203.2" y="66.04" size="1.27" layer="95" xref="yes"/>
-<pinref part="IC6" gate="G$1" pin="GPIO2"/>
-<wire x1="195.58" y1="66.04" x2="203.2" y2="66.04" width="0.1524" layer="91"/>
+<pinref part="IC6" gate="G$1" pin="GPIO4"/>
+<wire x1="195.58" y1="60.96" x2="203.2" y2="60.96" width="0.1524" layer="91"/>
+<label x="203.2" y="60.96" size="1.27" layer="95" xref="yes"/>
 </segment>
 </net>
@@
 <net name="WS2812_POWER" class="0">
 <segment>
-<wire x1="266.7" y1="66.04" x2="261.62" y2="66.04" width="0.1524" layer="91"/>
-<label x="261.62" y="66.04" size="1.27" layer="95" rot="R180" xref="yes"/>
-<pinref part="J2" gate="G$1" pin="2"/>
+<wire x1="281.94" y1="66.04" x2="284.48" y2="66.04" width="0.1524" layer="91"/>
+<label x="284.48" y="66.04" size="1.27" layer="95" xref="yes"/>
+<pinref part="J3" gate="G$1" pin="11"/>
 </segment>
 </net>
@@
 <wire x1="266.7" y1="55.88" x2="261.62" y2="55.88" width="0.1524" layer="91"/>
 <label x="261.62" y="55.88" size="1.27" layer="95" rot="R180" xref="yes"/>
-<pinref part="J2" gate="G$1" pin="6"/>
+<pinref part="J3" gate="G$1" pin="6"/>
 </segment>
 </net>
@@
 <wire x1="281.94" y1="55.88" x2="284.48" y2="55.88" width="0.1524" layer="91"/>
 <label x="284.48" y="55.88" size="1.27" layer="95" xref="yes"/>
-<pinref part="J2" gate="G$1" pin="7"/>
+<pinref part="J3" gate="G$1" pin="7"/>
 </segment>
 </net>
@@
 </segment>
 </net>
-<net name="CHRG_STAT" class="0">
-<segment>
-<pinref part="IC6" gate="G$1" pin="GPIO4"/>
-<wire x1="195.58" y1="60.96" x2="203.2" y2="60.96" width="0.1524" layer="91"/>
-<label x="203.2" y="60.96" size="1.27" layer="95" xref="yes"/>
-</segment>
-</net>
 <net name="3V3_SWITCHED" class="0">
 <segment>
 <wire x1="266.7" y1="68.58" x2="261.62" y2="68.58" width="0.1524" layer="91"/>
 <label x="261.62" y="68.58" size="1.27" layer="95" rot="R180" xref="yes"/>
-<pinref part="J2" gate="G$1" pin="1"/>
+<pinref part="J3" gate="G$1" pin="1"/>
 </segment>
 </net>
 <net name="EXTIO-0" class="0">
 <segment>
-<wire x1="266.7" y1="63.5" x2="261.62" y2="63.5" width="0.1524" layer="91"/>
-<label x="261.62" y="63.5" size="1.27" layer="95" rot="R180" xref="yes"/>
-<pinref part="J2" gate="G$1" pin="3"/>
+<wire x1="281.94" y1="63.5" x2="284.48" y2="63.5" width="0.1524" layer="91"/>
+<label x="284.48" y="63.5" size="1.27" layer="95" xref="yes"/>
+<pinref part="J3" gate="G$1" pin="10"/>
 </segment>
 <segment>
@@
 <net name="EXTIO-3" class="0">
 <segment>
-<wire x1="281.94" y1="60.96" x2="284.48" y2="60.96" width="0.1524" layer="91"/>
-<label x="284.48" y="60.96" size="1.27" layer="95" xref="yes"/>
-<pinref part="J2" gate="G$1" pin="9"/>
-</segment>
-<segment>
-<pinref part="IC6" gate="G$1" pin="GPIO5"/>
-<wire x1="195.58" y1="58.42" x2="200.66" y2="58.42" width="0.1524" layer="91"/>
-<label x="200.66" y="58.42" size="1.27" layer="95" xref="yes"/>
+<wire x1="266.7" y1="60.96" x2="261.62" y2="60.96" width="0.1524" layer="91"/>
+<label x="261.62" y="60.96" size="1.27" layer="95" rot="R180" xref="yes"/>
+<pinref part="J3" gate="G$1" pin="4"/>
+</segment>
+<segment>
+<pinref part="IC6" gate="G$1" pin="GPIO7"/>
+<wire x1="195.58" y1="53.34" x2="200.66" y2="53.34" width="0.1524" layer="91"/>
+<label x="200.66" y="53.34" size="1.27" layer="95" xref="yes"/>
 </segment>
 </net>
@@
 </segment>
 <segment>
-<wire x1="266.7" y1="60.96" x2="261.62" y2="60.96" width="0.1524" layer="91"/>
-<label x="261.62" y="60.96" size="1.27" layer="95" rot="R180" xref="yes"/>
-<pinref part="J2" gate="G$1" pin="4"/>
+<wire x1="281.94" y1="60.96" x2="284.48" y2="60.96" width="0.1524" layer="91"/>
+<label x="284.48" y="60.96" size="1.27" layer="95" xref="yes"/>
+<pinref part="J3" gate="G$1" pin="9"/>
 </segment>
 </net>
@@
 </segment>
 <segment>
-<wire x1="266.7" y1="58.42" x2="264.16" y2="58.42" width="0.1524" layer="91"/>
-<wire x1="264.16" y1="58.42" x2="261.62" y2="58.42" width="0.1524" layer="91"/>
-<label x="261.62" y="58.42" size="1.27" layer="95" rot="R180" xref="yes"/>
-<pinref part="J2" gate="G$1" pin="5"/>
+<wire x1="281.94" y1="58.42" x2="284.48" y2="58.42" width="0.1524" layer="91"/>
+<label x="284.48" y="58.42" size="1.27" layer="95" xref="yes"/>
+<pinref part="J3" gate="G$1" pin="8"/>
 </segment>
 </net>
@@
 </segment>
 <segment>
-<wire x1="281.94" y1="63.5" x2="284.48" y2="63.5" width="0.1524" layer="91"/>
-<label x="284.48" y="63.5" size="1.27" layer="95" xref="yes"/>
-<pinref part="J2" gate="G$1" pin="10"/>
+<wire x1="266.7" y1="63.5" x2="261.62" y2="63.5" width="0.1524" layer="91"/>
+<label x="261.62" y="63.5" size="1.27" layer="95" rot="R180" xref="yes"/>
+<pinref part="J3" gate="G$1" pin="3"/>
 </segment>
 </net>
 <net name="EXTIO-5" class="0">
 <segment>
-<pinref part="IC6" gate="G$1" pin="GPIO7"/>
-<wire x1="195.58" y1="53.34" x2="200.66" y2="53.34" width="0.1524" layer="91"/>
-<label x="200.66" y="53.34" size="1.27" layer="95" xref="yes"/>
-</segment>
-<segment>
-<wire x1="281.94" y1="66.04" x2="284.48" y2="66.04" width="0.1524" layer="91"/>
-<label x="284.48" y="66.04" size="1.27" layer="95" xref="yes"/>
-<pinref part="J2" gate="G$1" pin="11"/>
-</segment>
-</net>
-<net name="WS2812_POWER_EN" class="0">
+<wire x1="266.7" y1="66.04" x2="261.62" y2="66.04" width="0.1524" layer="91"/>
+<label x="261.62" y="66.04" size="1.27" layer="95" rot="R180" xref="yes"/>
+<pinref part="J3" gate="G$1" pin="2"/>
+</segment>
+<segment>
+<pinref part="IC6" gate="G$1" pin="GPIO5"/>
+<wire x1="195.58" y1="58.42" x2="200.66" y2="58.42" width="0.1524" layer="91"/>
+<label x="200.66" y="58.42" size="1.27" layer="95" xref="yes"/>
+</segment>
+</net>
+<net name="WS2812_DATA_OUT" class="0">
+<segment>
+<wire x1="266.7" y1="58.42" x2="261.62" y2="58.42" width="0.1524" layer="91"/>
+<label x="261.62" y="58.42" size="1.27" layer="95" rot="R180" xref="yes"/>
+<pinref part="J3" gate="G$1" pin="5"/>
+</segment>
+</net>
+<net name="CHRG_STAT" class="0">
 <segment>
 <label x="203.2" y="71.12" size="1.27" layer="95" xref="yes"/>
@@
 </segment>
 </net>
-<net name="WS2812_DATA_OUT" class="0">
-<segment>
-<pinref part="J2" gate="G$1" pin="8"/>
-<wire x1="281.94" y1="58.42" x2="284.48" y2="58.42" width="0.1524" layer="91"/>
-<label x="284.48" y="58.42" size="1.27" layer="95" xref="yes"/>
-</segment>
-</net>
+<net name="WS2812_POWER_EN" class="0">
+<segment>
+<label x="203.2" y="66.04" size="1.27" layer="95" xref="yes"/>
+<pinref part="IC6" gate="G$1" pin="GPIO2"/>
+<wire x1="195.58" y1="66.04" x2="203.2" y2="66.04" width="0.1524" layer="91"/>
+</segment>
+</net>
