File: sha2017_rev0_1_0_dev.sch (EAGLE design)
At the start: 203 parts, among them IC1 CP210X_USB_UART, IC2 AP7215, IC3 ESP32WROOM32, IC4 MCP73833, IC5 FXL6408, IC6 CPT112, Q1 MMBT2222A, Q2 MMBT2222A, Q3 MMBT2222A, Q4 MMBT2222A, Q5 SI1304 BDL, Q6 MMBT2222A, T1 BSS316N H6327, T2 BSS316N H6327, T3 BSS316N H6327, X2 2908-05WB-MG, X4 JST-PH3

Commit message: some more changes
Parts:
- F1, F2: value 500mA -> 900mA; PARTNO 0ZCJ0025FF2E -> (none)
- R23, R24: value 470R -> 4k7
- T1, T2, T3: value BSS316N H6327 -> MOSFET-PCHANNEL; PARTNO 726-BSS316NH6327XT -> (none)
Changed lines of the file:
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@@
 </part>
 <part name="GND46" library="supply1" deviceset="GND" device=""/>
-<part name="F1" library="SparkFun-PowerIC" deviceset="PTC" device="SMD" value="500mA">
-<attribute name="PARTNO" value="0ZCJ0025FF2E"/>
+<part name="F1" library="SparkFun-PowerIC" deviceset="PTC" device="SMD" value="900mA">
+<attribute name="PARTNO" value=""/>
 </part>
 <part name="D1" library="SparkFun-DiscreteSemi" deviceset="DIODE-SCHOTTKY" device="-PMEG4005EJ" value="SD05-7">
@@
 <attribute name="PARTNO" value="ERJ-3GEYJ103V"/>
 </part>
-<part name="F2" library="SparkFun-PowerIC" deviceset="PTC" device="SMD" value="500mA">
-<attribute name="PARTNO" value="0ZCJ0025FF2E"/>
+<part name="F2" library="SparkFun-PowerIC" deviceset="PTC" device="SMD" value="900mA">
+<attribute name="PARTNO" value=""/>
 </part>
 <part name="GND10" library="supply1" deviceset="GND" device=""/>
@@
 <attribute name="PARTNO" value="GRM188R71H104KA93D"/>
 </part>
-<part name="T1" library="SparkFun-DiscreteSemi" deviceset="MOSFET-PCHANNEL" device="" value="BSS316N H6327">
-<attribute name="PARTNO" value="726-BSS316NH6327XT"/>
+<part name="T1" library="SparkFun-DiscreteSemi" deviceset="MOSFET-PCHANNEL" device="" value="">
+<attribute name="PARTNO" value=""/>
 </part>
 <part name="R4" library="sha2017_rev0_1_0_dev" deviceset="R0603-DASHES" device="" value="10k">
@@
 <part name="U$1" library="badge" deviceset="MOTOR" device="10MM"/>
 <part name="P+7" library="supply1" deviceset="VCC" device=""/>
-<part name="R24" library="sha2017_rev0_1_0_dev" deviceset="R0603-DASHES" device="" value="470R">
-<attribute name="MF" value=""/>
-<attribute name="MPN" value=""/>
-<attribute name="OC_FARNELL" value="unknown"/>
-<attribute name="PARTNO" value="ERJ-3GEYJ103V"/>
-</part>
-<part name="R23" library="sha2017_rev0_1_0_dev" deviceset="R0603-DASHES" device="" value="470R">
+<part name="R24" library="sha2017_rev0_1_0_dev" deviceset="R0603-DASHES" device="" value="4k7">
+<attribute name="MF" value=""/>
+<attribute name="MPN" value=""/>
+<attribute name="OC_FARNELL" value="unknown"/>
+<attribute name="PARTNO" value="ERJ-3GEYJ103V"/>
+</part>
+<part name="R23" library="sha2017_rev0_1_0_dev" deviceset="R0603-DASHES" device="" value="4k7">
 <attribute name="MF" value=""/>
 <attribute name="MPN" value=""/>
@@
 <attribute name="PARTNO" value="GRM21BR61C475KA88K"/>
 </part>
-<part name="T2" library="SparkFun-DiscreteSemi" deviceset="MOSFET-PCHANNEL" device="" value="BSS316N H6327">
-<attribute name="PARTNO" value="726-BSS316NH6327XT"/>
-</part>
-<part name="T3" library="SparkFun-DiscreteSemi" deviceset="MOSFET-PCHANNEL" device="" value="BSS316N H6327">
-<attribute name="PARTNO" value="726-BSS316NH6327XT"/>
+<part name="T2" library="SparkFun-DiscreteSemi" deviceset="MOSFET-PCHANNEL" device="" value="">
+<attribute name="PARTNO" value=""/>
+</part>
+<part name="T3" library="SparkFun-DiscreteSemi" deviceset="MOSFET-PCHANNEL" device="" value="">
+<attribute name="PARTNO" value=""/>
 </part>
 <part name="TP1" library="SparkFun-Passives" deviceset="TEST-POINT" device="3">
