File: sha2017_rev1_0_0.sch (EAGLE design)
At the start: 198 parts, among them IC1 CP210X_USB_UART, IC2 AP7215, IC3 ESP32WROOM32, IC4 TP4056, M1 MOTOR10MM, Q3 MMBT2222A, Q4 MMBT2222A, Q5 SI1304 BDL, T1 MOSFET-PCHANNEL, T2 AO3400, T3 MOSFET-PCHANNEL, T4 AO3400, U1 MPR121QR2, X2 2908-05WB-MG, X4 JST-PH3

Commit message: Fix schematic
Parts:
- removed T4: AO3400, zetex:NMOSSOT23
- added Q1, Q2, Q6: MMBT2222A, SparkFun-DiscreteSemi:TRANSISTOR_NPNMMBT2222A
- added R27: 10k, 00ralf:R0603-DASHES
- R10: value 470 -> 10k
- R11, R28, R4, R9: value 100k -> 10k
- T2: value AO3400 -> MOSFET-PCHANNEL; device zetex:NMOSSOT23 -> SparkFun-DiscreteSemi:MOSFET-PCHANNEL
Connections:
- removed net PERIPHERAL_POWER_EN: R9.1, T2.G, U1.ELE4
- removed net SD_POWER_EN: D100.VSS, D101.VSS, D102.VSS, D103.VSS, D104.VSS, D105.VSS, R28.1, T2.D, T3.G
- new net N$17: Q6.C, R28.1, T3.G
- new net N$45: Q2.B, R11.1
- new net N$52: Q1.B, R10.2
- new net N$53: Q1.C, R9.1, T2.G
- new net WS2812_POWER: C1.2, C13.1, C2.2, C3.2, C4.2, C5.2, C6.2, D100.VDD, D101.VDD, D102.VDD, D103.VDD, D104.VDD, D105.VDD, T2.D, TP117.1, X3.11
- new net WS2812_POWER_EN: R10.1, R27.1, U1.ELE4
- net GND: now also D100.VSS, D101.VSS, D102.VSS, D103.VSS, D104.VSS, D105.VSS, Q1.E, Q2.E, Q6.E; no longer R11.2, R9.2, T2.S, T4.S
- net N$15: now also Q6.B, R27.2; no longer D105.DIN, R10.1
- net N$16: now also Q2.C; no longer T4.D
- net VCC: now also R9.2, T2.S; no longer C1.2, C13.1, C2.2, C3.2, C4.2, C5.2, C6.2, D100.VDD, D101.VDD, D102.VDD, D103.VDD, D104.VDD, D105.VDD, TP117.1, X3.11
- net VIBRATOR: now also R11.2; no longer R11.1, T4.G
- net WS2812_DATA: now also D105.DIN; no longer R10.2
Other:
- moved on the sheet: C1, C13, C2, C3, C4, C5, C6, D100, D101, D102, D103, D104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

Commit message: MarkusBec rerouting and fixes
Parts:
- R30: value 150k -> 0R27; device sha2017_rev0_1_0_dev:R0603-DASHES -> rcl:R-EU_R1206
Connections:
- removed net N$56: TOUCH_SEL.RIGHT, U1.ELE1
- new net N$48: TOUCH_SEL.RIGHT, U1.ELE5
- net CHRG_STAT: now also U1.ELE9; no longer U1.ELE6
- net N$1: now also TOUCH_B.P$1, U1.ELE1; no longer TOUCH_A.P$1, U1.ELE8
- net N$24: now also TOUCH_START.P$1, U1.ELE2; no longer TOUCH_B.P$1, U1.ELE9
- net N$25: now also TOUCH_SELECT.P$1; no longer TOUCH_SEL.LEFT
- net N$44: now also U1.ELE4; no longer U1.ELE0
- net N$46: now also TOUCH_SEL.LEFT, U1.ELE7; no longer TOUCH_SELECT.P$1, U1.ELE10
- net N$47: now also U1.ELE6; no longer U1.ELE2
- net N$6: now also TOUCH_A.P$1, U1.ELE0; no longer TOUCH_START.P$1, U1.ELE11
- net SD_CD: now also U1.ELE11; no longer U1.ELE5
- net VIBRATOR: now also U1.ELE8; no longer U1.ELE7
- net WS2812_POWER_EN: now also U1.ELE10; no longer U1.ELE4
Other:
- moved on the sheet: TOUCH_A, TOUCH_B, TOUCH_SEL, TOUCH_SELECT, TOUCH_START
Changed lines of the file:
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@@
 <part name="+3V7" library="supply1" deviceset="+3V3" device=""/>
 <part name="U1" library="Freescale_By_element14_Batch_1" deviceset="MPR121QR2" device=""/>
-<part name="R30" library="sha2017_rev0_1_0_dev" deviceset="R0603-DASHES" device="" value="150k">
+<part name="R30" library="rcl" deviceset="R-EU_" device="R1206" value="0R27">
 <attribute name="PARTNO" value="ERJ-3GEYJ154V"/>
 </part>
@@
 <attribute name="PARTNO" x="72.39" y="212.09" size="1.778" layer="96" rot="MR0" display="off"/>
 </instance>
-<instance part="TOUCH_A" gate="G$1" x="157.48" y="48.26" rot="R270">
+<instance part="TOUCH_A" gate="G$1" x="170.18" y="48.26" rot="R270">
+<attribute name="PARTNO" x="170.18" y="48.26" size="5.08" layer="96" display="off"/>
+</instance>
+<instance part="TOUCH_B" gate="G$1" x="157.48" y="48.26" rot="R270">
 <attribute name="PARTNO" x="157.48" y="48.26" size="5.08" layer="96" display="off"/>
 </instance>
-<instance part="TOUCH_B" gate="G$1" x="142.24" y="50.8" rot="R270">
-<attribute name="PARTNO" x="142.24" y="50.8" size="5.08" layer="96" display="off"/>
-</instance>
-<instance part="TOUCH_SEL" gate="G$1" x="177.8" y="93.98">
-<attribute name="PARTNO" x="177.8" y="93.98" size="5.08" layer="96" display="off"/>
+<instance part="TOUCH_SEL" gate="G$1" x="190.5" y="96.52">
+<attribute name="PARTNO" x="190.5" y="96.52" size="5.08" layer="96" display="off"/>
 </instance>
 <instance part="+3V4" gate="G$1" x="15.24" y="53.34" rot="R90"/>
@@
 <instance part="+2V4" gate="G$1" x="208.28" y="76.2"/>
 <instance part="+2V5" gate="G$1" x="200.66" y="76.2"/>
-<instance part="TOUCH_SELECT" gate="G$1" x="124.46" y="55.88" rot="R270"/>
-<instance part="TOUCH_START" gate="G$1" x="109.22" y="58.42" rot="R270"/>
+<instance part="TOUCH_SELECT" gate="G$1" x="132.08" y="48.26" rot="R270"/>
+<instance part="TOUCH_START" gate="G$1" x="144.78" y="48.26" rot="R270"/>
 <instance part="R1" gate="G$1" x="58.42" y="96.52" rot="R90">
 <attribute name="PARTNO" x="58.42" y="96.52" size="5.08" layer="96" display="off"/>
@@
 </segment>
 <segment>
-<label x="109.22" y="78.74" size="1.27" layer="95" xref="yes"/>
-<wire x1="104.14" y1="78.74" x2="109.22" y2="78.74" width="0.1524" layer="91"/>
-<pinref part="U1" gate="A" pin="ELE6"/>
+<label x="111.76" y="71.12" size="1.27" layer="95" xref="yes"/>
+<wire x1="104.14" y1="71.12" x2="111.76" y2="71.12" width="0.1524" layer="91"/>
+<pinref part="U1" gate="A" pin="ELE9"/>
 </segment>
 </net>
@@
 </segment>
 <segment>
-<label x="106.68" y="83.82" size="1.27" layer="95" xref="yes"/>
-<wire x1="104.14" y1="83.82" x2="106.68" y2="83.82" width="0.1524" layer="91"/>
-<pinref part="U1" gate="A" pin="ELE4"/>
+<label x="111.76" y="68.58" size="1.27" layer="95" xref="yes"/>
+<wire x1="104.14" y1="68.58" x2="111.76" y2="68.58" width="0.1524" layer="91"/>
+<pinref part="U1" gate="A" pin="ELE10"/>
 </segment>
 </net>
@@
 <pinref part="D105" gate="G$1" pin="DOUT"/>
 <wire x1="265.43" y1="214.63" x2="273.05" y2="214.63" width="0.1524" layer="91"/>
-</segment>
-</net>
-<net name="N$56" class="3">
-<segment>
-<pinref part="TOUCH_SEL" gate="G$1" pin="RIGHT"/>
-<wire x1="187.96" y1="78.74" x2="187.96" y2="93.98" width="0.1524" layer="91"/>
-<wire x1="160.02" y1="78.74" x2="187.96" y2="78.74" width="0.1524" layer="91"/>
-<wire x1="160.02" y1="78.74" x2="160.02" y2="91.44" width="0.1524" layer="91"/>
-<pinref part="U1" gate="A" pin="ELE1"/>
-<wire x1="104.14" y1="91.44" x2="160.02" y2="91.44" width="0.1524" layer="91"/>
 </segment>
 </net>
@@
 <label x="287.02" y="76.2" size="1.27" layer="95" xref="yes"/>
 <pinref part="X3" gate="G$1" pin="7"/>
-</segment>
-</net>
-<net name="N$25" class="3">
-<segment>
-<pinref part="TOUCH_SEL" gate="G$1" pin="LEFT"/>
-<pinref part="U1" gate="A" pin="ELE3"/>
-<wire x1="104.14" y1="86.36" x2="165.1" y2="86.36" width="0.1524" layer="91"/>
-<wire x1="165.1" y1="86.36" x2="165.1" y2="93.98" width="0.1524" layer="91"/>
-<wire x1="165.1" y1="93.98" x2="167.64" y2="93.98" width="0.1524" layer="91"/>
 </segment>
 </net>
@@
 <net name="SD_CD" class="0">
 <segment>
-<label x="106.68" y="81.28" size="1.27" layer="95" xref="yes"/>
-<wire x1="104.14" y1="81.28" x2="106.68" y2="81.28" width="0.1524" layer="91"/>
-<pinref part="U1" gate="A" pin="ELE5"/>
+<label x="111.76" y="66.04" size="1.27" layer="95" xref="yes"/>
+<pinref part="U1" gate="A" pin="ELE11"/>
+<wire x1="111.76" y1="66.04" x2="104.14" y2="66.04" width="0.1524" layer="91"/>
 </segment>
 </net>
 <net name="VIBRATOR" class="0">
 <segment>
-<label x="109.22" y="76.2" size="1.27" layer="95" xref="yes"/>
-<wire x1="104.14" y1="76.2" x2="109.22" y2="76.2" width="0.1524" layer="91"/>
-<pinref part="U1" gate="A" pin="ELE7"/>
+<label x="111.76" y="73.66" size="1.27" layer="95" xref="yes"/>
+<wire x1="104.14" y1="73.66" x2="111.76" y2="73.66" width="0.1524" layer="91"/>
+<pinref part="U1" gate="A" pin="ELE8"/>
 </segment>
 </net>
@@
 <segment>
 <pinref part="TOUCH_SEL" gate="G$1" pin="DOWN"/>
-<wire x1="177.8" y1="81.28" x2="177.8" y2="83.82" width="0.1524" layer="91"/>
-<wire x1="177.8" y1="81.28" x2="162.56" y2="81.28" width="0.1524" layer="91"/>
-<wire x1="162.56" y1="81.28" x2="162.56" y2="93.98" width="0.1524" layer="91"/>
-<wire x1="162.56" y1="93.98" x2="104.14" y2="93.98" width="0.1524" layer="91"/>
-<pinref part="U1" gate="A" pin="ELE0"/>
-</segment>
-</net>
-<net name="N$1" class="3">
-<segment>
-<pinref part="TOUCH_A" gate="G$1" pin="P$1"/>
-<wire x1="157.48" y1="73.66" x2="157.48" y2="55.88" width="0.1524" layer="91"/>
-<pinref part="U1" gate="A" pin="ELE8"/>
-<wire x1="104.14" y1="73.66" x2="157.48" y2="73.66" width="0.1524" layer="91"/>
-</segment>
-</net>
-<net name="N$47" class="3">
-<segment>
-<pinref part="TOUCH_SEL" gate="G$1" pin="UP"/>
-<wire x1="157.48" y1="104.14" x2="177.8" y2="104.14" width="0.1524" layer="91"/>
-<wire x1="157.48" y1="104.14" x2="157.48" y2="88.9" width="0.1524" layer="91"/>
-<pinref part="U1" gate="A" pin="ELE2"/>
-<wire x1="104.14" y1="88.9" x2="157.48" y2="88.9" width="0.1524" layer="91"/>
-</segment>
-</net>
-<net name="N$6" class="3">
-<segment>
-<pinref part="U1" gate="A" pin="ELE11"/>
-<pinref part="TOUCH_START" gate="G$1" pin="P$1"/>
-<wire x1="104.14" y1="66.04" x2="109.22" y2="66.04" width="0.1524" layer="91"/>
-</segment>
-</net>
-<net name="N$46" class="3">
-<segment>
-<pinref part="U1" gate="A" pin="ELE10"/>
-<pinref part="TOUCH_SELECT" gate="G$1" pin="P$1"/>
-<wire x1="104.14" y1="68.58" x2="124.46" y2="68.58" width="0.1524" layer="91"/>
-<wire x1="124.46" y1="68.58" x2="124.46" y2="63.5" width="0.1524" layer="91"/>
-</segment>
-</net>
-<net name="N$24" class="3">
-<segment>
-<pinref part="U1" gate="A" pin="ELE9"/>
-<pinref part="TOUCH_B" gate="G$1" pin="P$1"/>
-<wire x1="104.14" y1="71.12" x2="142.24" y2="71.12" width="0.1524" layer="91"/>
-<wire x1="142.24" y1="71.12" x2="142.24" y2="58.42" width="0.1524" layer="91"/>
+<pinref part="U1" gate="A" pin="ELE4"/>
+<wire x1="104.14" y1="83.82" x2="190.5" y2="83.82" width="0.1524" layer="91"/>
+<wire x1="190.5" y1="83.82" x2="190.5" y2="86.36" width="0.1524" layer="91"/>
 </segment>
 </net>
@@
 </segment>
 </net>
+<net name="N$6" class="3">
+<segment>
+<pinref part="TOUCH_A" gate="G$1" pin="P$1"/>
+<wire x1="170.18" y1="93.98" x2="170.18" y2="55.88" width="0.1524" layer="91"/>
+<pinref part="U1" gate="A" pin="ELE0"/>
+<wire x1="104.14" y1="93.98" x2="170.18" y2="93.98" width="0.1524" layer="91"/>
+</segment>
+</net>
+<net name="N$1" class="3">
+<segment>
+<pinref part="U1" gate="A" pin="ELE1"/>
+<pinref part="TOUCH_B" gate="G$1" pin="P$1"/>
+<wire x1="104.14" y1="91.44" x2="157.48" y2="91.44" width="0.1524" layer="91"/>
+<wire x1="157.48" y1="91.44" x2="157.48" y2="55.88" width="0.1524" layer="91"/>
+</segment>
+</net>
+<net name="N$24" class="3">
+<segment>
+<pinref part="U1" gate="A" pin="ELE2"/>
+<pinref part="TOUCH_START" gate="G$1" pin="P$1"/>
+<wire x1="104.14" y1="88.9" x2="144.78" y2="88.9" width="0.1524" layer="91"/>
+<wire x1="144.78" y1="88.9" x2="144.78" y2="55.88" width="0.1524" layer="91"/>
+</segment>
+</net>
+<net name="N$25" class="3">
+<segment>
+<pinref part="U1" gate="A" pin="ELE3"/>
+<pinref part="TOUCH_SELECT" gate="G$1" pin="P$1"/>
+<wire x1="104.14" y1="86.36" x2="132.08" y2="86.36" width="0.1524" layer="91"/>
+<wire x1="132.08" y1="86.36" x2="132.08" y2="55.88" width="0.1524" layer="91"/>
+</segment>
+</net>
+<net name="N$46" class="3">
+<segment>
+<pinref part="U1" gate="A" pin="ELE7"/>
+<pinref part="TOUCH_SEL" gate="G$1" pin="LEFT"/>
+<wire x1="104.14" y1="76.2" x2="180.34" y2="76.2" width="0.1524" layer="91"/>
+<wire x1="180.34" y1="76.2" x2="180.34" y2="96.52" width="0.1524" layer="91"/>
+</segment>
+</net>
+<net name="N$47" class="3">
+<segment>
+<pinref part="U1" gate="A" pin="ELE6"/>
+<wire x1="104.14" y1="78.74" x2="177.8" y2="78.74" width="0.1524" layer="91"/>
+<wire x1="177.8" y1="78.74" x2="177.8" y2="109.22" width="0.1524" layer="91"/>
+<pinref part="TOUCH_SEL" gate="G$1" pin="UP"/>
+<wire x1="177.8" y1="109.22" x2="190.5" y2="109.22" width="0.1524" layer="91"/>
+<wire x1="190.5" y1="109.22" x2="190.5" y2="106.68" width="0.1524" layer="91"/>
+</segment>
+</net>
+<net name="N$48" class="3">
+<segment>
+<pinref part="U1" gate="A" pin="ELE5"/>
+<wire x1="104.14" y1="81.28" x2="175.26" y2="81.28" width="0.1524" layer="91"/>
+<wire x1="175.26" y1="81.28" x2="175.26" y2="111.76" width="0.1524" layer="91"/>
+<pinref part="TOUCH_SEL" gate="G$1" pin="RIGHT"/>
+<wire x1="175.26" y1="111.76" x2="200.66" y2="111.76" width="0.1524" layer="91"/>
+<wire x1="200.66" y1="111.76" x2="200.66" y2="96.52" width="0.1524" layer="91"/>
+</segment>
+</net>

Commit message: R2 0603->1206
Parts:
- R2: device 00ralf:R0603-DASHES -> resistor:R-EU_R1206
Changed lines of the file:
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@@
 <grid distance="0.1" unitdist="inch" unit="inch" style="lines" multiple="1" display="no" altdistance="0.01" altunitdist="inch" altunit="inch"/>
 <layers>
-<layer number="1" name="Top" color="4" fill="1" visible="no" active="no"/>
-<layer number="2" name="Route2" color="1" fill="3" visible="no" active="no"/>
-<layer number="3" name="Route3" color="4" fill="3" visible="no" active="no"/>
-<layer number="4" name="Route4" color="1" fill="4" visible="no" active="no"/>
-<layer number="5" name="Route5" color="4" fill="4" visible="no" active="no"/>
-<layer number="6" name="Route6" color="1" fill="8" visible="no" active="no"/>
-<layer number="7" name="Route7" color="4" fill="8" visible="no" active="no"/>
-<layer number="8" name="Route8" color="1" fill="2" visible="no" active="no"/>
-<layer number="9" name="Route9" color="4" fill="2" visible="no" active="no"/>
-<layer number="10" name="Route10" color="1" fill="7" visible="no" active="no"/>
-<layer number="11" name="Route11" color="4" fill="7" visible="no" active="no"/>
-<layer number="12" name="Route12" color="1" fill="5" visible="no" active="no"/>
-<layer number="13" name="Route13" color="4" fill="5" visible="no" active="no"/>
-<layer number="14" name="Route14" color="1" fill="6" visible="no" active="no"/>
-<layer number="15" name="Route15" color="4" fill="6" visible="no" active="no"/>
-<layer number="16" name="Bottom" color="1" fill="1" visible="no" active="no"/>
-<layer number="17" name="Pads" color="2" fill="1" visible="no" active="no"/>
-<layer number="18" name="Vias" color="2" fill="1" visible="no" active="no"/>
-<layer number="19" name="Unrouted" color="6" fill="1" visible="no" active="no"/>
-<layer number="20" name="Dimension" color="15" fill="1" visible="no" active="no"/>
-<layer number="21" name="tPlace" color="7" fill="1" visible="no" active="no"/>
-<layer number="22" name="bPlace" color="7" fill="1" visible="no" active="no"/>
-<layer number="23" name="tOrigins" color="15" fill="1" visible="no" active="no"/>
-<layer number="24" name="bOrigins" color="15" fill="1" visible="no" active="no"/>
-<layer number="25" name="tNames" color="7" fill="1" visible="no" active="no"/>
-<layer number="26" name="bNames" color="7" fill="1" visible="no" active="no"/>
-<layer number="27" name="tValues" color="7" fill="1" visible="no" active="no"/>
-<layer number="28" name="bValues" color="7" fill="1" visible="no" active="no"/>
+<layer number="1" name="Top" color="4" fill="1" visible="yes" active="no"/>
+<layer number="2" name="Route2" color="1" fill="3" visible="yes" active="no"/>
+<layer number="3" name="Route3" color="4" fill="3" visible="yes" active="no"/>
+<layer number="4" name="Route4" color="1" fill="4" visible="yes" active="no"/>
+<layer number="5" name="Route5" color="4" fill="4" visible="yes" active="no"/>
+<layer number="6" name="Route6" color="1" fill="8" visible="yes" active="no"/>
+<layer number="7" name="Route7" color="4" fill="8" visible="yes" active="no"/>
+<layer number="8" name="Route8" color="1" fill="2" visible="yes" active="no"/>
+<layer number="9" name="Route9" color="4" fill="2" visible="yes" active="no"/>
+<layer number="10" name="Route10" color="1" fill="7" visible="yes" active="no"/>
+<layer number="11" name="Route11" color="4" fill="7" visible="yes" active="no"/>
+<layer number="12" name="Route12" color="1" fill="5" visible="yes" active="no"/>
+<layer number="13" name="Route13" color="4" fill="5" visible="yes" active="no"/>
+<layer number="14" name="Route14" color="1" fill="6" visible="yes" active="no"/>
+<layer number="15" name="Route15" color="4" fill="6" visible="yes" active="no"/>
+<layer number="16" name="Bottom" color="1" fill="1" visible="yes" active="no"/>
+<layer number="17" name="Pads" color="2" fill="1" visible="yes" active="no"/>
+<layer number="18" name="Vias" color="2" fill="1" visible="yes" active="no"/>
+<layer number="19" name="Unrouted" color="6" fill="1" visible="yes" active="no"/>
+<layer number="20" name="Dimension" color="15" fill="1" visible="yes" active="no"/>
+<layer number="21" name="tPlace" color="7" fill="1" visible="yes" active="no"/>
+<layer number="22" name="bPlace" color="7" fill="1" visible="yes" active="no"/>
+<layer number="23" name="tOrigins" color="15" fill="1" visible="yes" active="no"/>
+<layer number="24" name="bOrigins" color="15" fill="1" visible="yes" active="no"/>
+<layer number="25" name="tNames" color="7" fill="1" visible="yes" active="no"/>
+<layer number="26" name="bNames" color="7" fill="1" visible="yes" active="no"/>
+<layer number="27" name="tValues" color="7" fill="1" visible="yes" active="no"/>
+<layer number="28" name="bValues" color="7" fill="1" visible="yes" active="no"/>
 <layer number="29" name="tStop" color="7" fill="3" visible="no" active="no"/>
 <layer number="30" name="bStop" color="7" fill="6" visible="no" active="no"/>
@@
 <layer number="35" name="tGlue" color="7" fill="4" visible="no" active="no"/>
 <layer number="36" name="bGlue" color="7" fill="5" visible="no" active="no"/>
-<layer number="37" name="tTest" color="7" fill="1" visible="no" active="no"/>
-<layer number="38" name="bTest" color="7" fill="1" visible="no" active="no"/>
+<layer number="37" name="tTest" color="7" fill="1" visible="yes" active="no"/>
+<layer number="38" name="bTest" color="7" fill="1" visible="yes" active="no"/>
 <layer number="39" name="tKeepout" color="4" fill="11" visible="no" active="no"/>
 <layer number="40" name="bKeepout" color="1" fill="11" visible="no" active="no"/>
@@
 <layer number="44" name="Drills" color="7" fill="1" visible="no" active="no"/>
 <layer number="45" name="Holes" color="7" fill="1" visible="no" active="no"/>
-<layer number="46" name="Milling" color="3" fill="1" visible="no" active="no"/>
-<layer number="47" name="Measures" color="7" fill="1" visible="no" active="no"/>
-<layer number="48" name="Document" color="7" fill="1" visible="no" active="no"/>
-<layer number="49" name="Reference" color="7" fill="1" visible="no" active="no"/>
-<layer number="50" name="dxf" color="7" fill="1" visible="no" active="no"/>
-<layer number="51" name="tDocu" color="7" fill="1" visible="no" active="no"/>
-<layer number="52" name="bDocu" color="7" fill="1" visible="no" active="no"/>
-<layer number="53" name="tGND_GNDA" color="7" fill="9" visible="no" active="no"/>
-<layer number="54" name="bGND_GNDA" color="1" fill="9" visible="no" active="no"/>
-<layer number="56" name="wert" color="7" fill="1" visible="no" active="no"/>
-<layer number="57" name="tCAD" color="7" fill="1" visible="no" active="no"/>
-<layer number="58" name="bCAD" color="11" fill="1" visible="no" active="no"/>
-<layer number="59" name="tCarbon" color="7" fill="1" visible="no" active="no"/>
-<layer number="60" name="bCarbon" color="7" fill="1" visible="no" active="no"/>
-<layer number="61" name="stand" color="7" fill="1" visible="no" active="no"/>
+<layer number="46" name="Milling" color="3" fill="1" visible="yes" active="no"/>
+<layer number="47" name="Measures" color="7" fill="1" visible="yes" active="no"/>
+<layer number="48" name="Document" color="7" fill="1" visible="yes" active="no"/>
+<layer number="49" name="Reference" color="7" fill="1" visible="yes" active="no"/>
+<layer number="50" name="dxf" color="7" fill="1" visible="yes" active="no"/>
+<layer number="51" name="tDocu" color="7" fill="1" visible="yes" active="no"/>
+<layer number="52" name="bDocu" color="7" fill="1" visible="yes" active="no"/>
+<layer number="53" name="tGND_GNDA" color="7" fill="9" visible="yes" active="no"/>
+<layer number="54" name="bGND_GNDA" color="1" fill="9" visible="yes" active="no"/>
+<layer number="56" name="wert" color="7" fill="1" visible="yes" active="no"/>
+<layer number="57" name="tCAD" color="7" fill="1" visible="yes" active="no"/>
+<layer number="58" name="bCAD" color="11" fill="1" visible="yes" active="no"/>
+<layer number="59" name="tCarbon" color="7" fill="1" visible="yes" active="no"/>
+<layer number="60" name="bCarbon" color="7" fill="1" visible="yes" active="no"/>
+<layer number="61" name="stand" color="7" fill="1" visible="yes" active="no"/>
 <layer number="90" name="Modules" color="5" fill="1" visible="yes" active="yes"/>
 <layer number="91" name="Nets" color="2" fill="1" visible="yes" active="yes"/>
@@
 </part>
 <part name="GND1" library="supply1" deviceset="GND" device=""/>
-<part name="R2" library="00ralf" deviceset="R0603-DASHES" device="" value="27R">
+<part name="R2" library="resistor" deviceset="R-EU_" device="R1206" value="27R">
 <attribute name="PARTNO" value="ERJ-3GEYJ220V"/>
 </part>
